File: KiCAD/MIX04/MIX04.kicad_pcb (KiCad board)
At the start: 2 copper layers, 66 x 99.1 mm, 45 parts, among them J1 IN1, J2 INV_OUT, J3 IN2, J4 OUT, J5 IN3, J6 IN4, J7 ERK_PWR, J8 TP_GND, U1 NJM4580, U2 NJM4580

Commit message: Board design
Parts:
- added G***: LOGO, myfootprint:Silk_PNPN_Manufactory_600dpi, F.Cu at (113.4, 73.6)
- moved C3 3.81 mm to (161.3, 139.7), turned to 0 degrees
- moved D1 2.54 mm to (114.9, 90.2), turned to 180 degrees
Routing:
- net Net-(J6-Pad1): track 0.00 -> 114.3 mm
- net +12V: track 2.54 -> 94.5 mm
- net Net-(C3-Pad1): track 0.00 -> 86.6 mm
- net Net-(C2-Pad2): track 0.00 -> 85.2 mm
- net Net-(J5-Pad1): track 0.00 -> 82.0 mm
- net Net-(C2-Pad1): track 0.00 -> 71.1 mm
- net -12V: track 0.00 -> 63.3 mm
- net Net-(J3-Pad1): track 0.00 -> 49.8 mm
- net Net-(C3-Pad2): track 0.00 -> 49.5 mm
- net Net-(C1-Pad1): track 0.00 -> 41.1 mm
- net Net-(J1-Pad1): track 0.00 -> 16.5 mm
- net Net-(D2-Pad1): track 0.00 -> 10.2 mm
- net Net-(D1-Pad2): track 0.00 -> 10.2 mm
- net Net-(C1-Pad2): track 0.00 -> 9.54 mm
- net Net-(R4-Pad1): track 0.00 -> 5.11 mm
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- added copper zone on B.Cu, net GND
Other:
- board text added: "G INV_OUT"
- board text added: "G OUT"
- board text added: "GND"
- board text added: "IN1 G"
- board text added: "IN1 LVL"
- board text added: "IN2 G"
- board text added: "IN2 LVL"
- board text added: "IN3 G"
- board text added: "IN3 LVL"
- board text added: "IN4 G"
- board text added: "IN4 LVL"
- board text added: "MIX04 Ver.1.0"
- board text added: "OUT LVL"
- board text added: "V- G G G V+"
- board text added: "https://dad8893.blogspot.com/"

Commit message: Panel design
Parts:
- moved C3 40.0 mm to (142.9, 104.1), turned to 270 degrees
- moved H2 1.27 mm to (163.8, 50.8)
- moved H4 1.27 mm to (163.8, 144.8)
- moved G*** 0.30 mm to (113.3, 73.9)
Routing:
- net Net-(C3-Pad2): track 49.5 -> 44.5 mm
- net Net-(C3-Pad1): track 86.6 -> 83.3 mm
Other:
- board size 66 x 99.1 mm -> 64.8 x 99.1 mm
